File: Projects/2016/MIDIBots/kicad/MIDI_Shield.sch (KiCad schematic (older format))
At the start: 12 parts, among them IC1 PC900V, P1 MIDI_IN, P2 MIDI_THRU, SW1 SW_PUSHBUTTON, SW2 DIPS_04, U1 74HC14

Commit message: Various corrections, tidying, and TODO updates for the MIDI shield schematic
Parts:
- added D?: LED, symbol LED
- added R?: 1K, symbol R
- added RV?: 10K, symbol POT
- added SW?: SW_PUSHBUTTON, symbol SW_PUSHBUTTON
- D1: value DIODE -> 1N914
Connections:
- net labels added: LATENCY_ADJ, LED
- wire segments 29 -> 43
- no-connect marks 16 -> 14
Other:
- note added: "Arduino shield"
- note added: "MIDI input"
- note added: "MIDI thru"
- note added: "Power"
- note added: "TODO: I should probably have used proper power ports from the beginning, rather than labelled ports."
- note added: "TODO: IIRC there was another pot planned"
- note added: "TODO: series resistor?"
- note added: "TODO: switch debouncing?"
- note added: "TODO:\n\n[ ] Servo output(s)\n[ ] MOSFET output(s)\n[ ] RX disconnection switch\n[ ] DIN connector grounding (pin 2, one end only? cap? what about chassis ground?)\n[ ] EMI ferrite beads on I/O lines?\n\n[X] 12 V connector (incl. GND)? Just use Arduino barrel jack.\n\n[Y] Reset switch\n[Y] MIDI THRU circuitry (buffer)\n[Y] Self-test button\n[Y] Latency control potentiometer\n[Y] LED + resistor on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"
- note added: "User interface"
- note removed: "TODO:\n[ ] LED + resistor on Pin 13\n[ ] Servo output(s)\n[ ] MOSFET output(s)\n[ ] RX disconnection switch\n[ ] MIDI THRU circuitry (buffer)\n[ ] 12 V connector (incl. GND)? Or just use Arduino barrel jack?\n\n"
- moved on the sheet: SHIELD1, SW1, SW2

Commit message: Added some grounds and N/Cs for the DIN connectors
Connections:
- wire segments 43 -> 40
- no-connect marks 14 -> 18
Other:
- note added: "Do we need all these GND labels?\nWon't the parent Arduino board connect these anyway?"
Changed lines of the file:
@@
 	7250 4250 7250 4350
 Wire Wire Line
-	7250 4350 7350 4350
-Wire Wire Line
-	7350 4350 7400 4350
-Wire Wire Line
-	7400 4350 7450 4350
-Wire Wire Line
-	7450 4350 7550 4350
+	7250 4350 7550 4350
 Wire Wire Line
 	7550 4350 7550 4250
@@
 NoConn ~ 3900 5600
 Wire Wire Line
-	3050 1450 3150 1450
-Wire Wire Line
-	3150 1450 3350 1450
+	3050 1450 3350 1450
 Wire Wire Line
 	2400 1450 2550 1450
 Wire Wire Line
-	3350 1650 3350 1850
-Wire Wire Line
-	3350 1850 3150 1850
-Wire Wire Line
-	3150 1850 2400 1850
+	3350 1850 3350 1650
+Wire Wire Line
+	2400 1850 3350 1850
 Wire Wire Line
 	2400 1850 2400 1650
@@
 	4050 1050 4050 1450
 Wire Wire Line
-	4050 1550 4600 1550
+	4050 1550 5100 1550
 Text Label 4600 950  2    60   ~ 0
 +5V
@@
 Text Notes 6800 2050 0    60   ~ 0
 TODO:\n\n[ ] Servo output(s)\n[ ] MOSFET output(s)\n[ ] RX disconnection switch\n[ ] DIN connector grounding (pin 2, one end only? cap? what about chassis ground?)\n[ ] EMI ferrite beads on I/O lines?\n\n[X] 12 V connector (incl. GND)? Just use Arduino barrel jack.\n\n[Y] Reset switch\n[Y] MIDI THRU circuitry (buffer)\n[Y] Self-test button\n[Y] Latency control potentiometer\n[Y] LED + resistor on Pin 13\n
-Text Label 4600 1550 0    60   ~ 0
+Text Label 5100 1550 0    60   ~ 0
 MIDI_IN_TTL
 Text Label 3900 5800 0    60   ~ 0
@@
 Connection ~ 3150 1450
 Connection ~ 3150 1850
+Text Notes 2400 6200 0    60   ~ 0
+Do we need all these GND labels?\nWon't the parent Arduino board connect these anyway?
+$Comp
+L GND #PWR?
+U 1 1 572B0D3F
+P 5500 3300
+F 0 "#PWR?" H 5500 3300 30  0001 C CNN
+F 1 "GND" H 5500 3230 30  0001 C CNN
+F 2 "" H 5500 3300 60  0000 C CNN
+F 3 "" H 5500 3300 60  0000 C CNN
+	1    5500 3300
+	1    0    0    -1
+$EndComp
+NoConn ~ 5200 3000
+NoConn ~ 4600 2400
+Wire Wire Line
+	5200 2800 5500 2800
+Wire Wire Line
+	5500 2800 5500 3300
+NoConn ~ 1200 1650
+NoConn ~ 1800 1050
+Connection ~ 4600 1550
 $EndSCHEMATC

Commit message: Amended pin functions and updated KiCAD schematic to match
Parts:
- gave numbers to parts that had none: 4
Connections:
- net labels added: MIDI_OUT_TTL, MOSFET, MOSFET_PWM, SERVO_1, SERVO_2, SERVO_3, STEPPER_DIR, STEPPER_STEP
- wire segments 40 -> 36
- no-connect marks 18 -> 10
Other:
- note added: "TODO:\n\n[ ] Servo output(s)\n[ ] MOSFET output(s)\n[ ] RX disconnection switch\n[ ] DIN connector grounding (pin 2, one end only? cap? what about chassis ground?)\n[ ] EMI ferrite beads on I/O lines?\n[ ] Polarised SIL connectors for MIDI I/O\n\n[X] 12 V connector (incl. GND)? Just use Arduino barrel jack.\n\n[Y] Reset switch\n[Y] MIDI THRU circuitry (buffer)\n[Y] Self-test button\n[Y] Latency c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"
- note removed: "TODO:\n\n[ ] Servo output(s)\n[ ] MOSFET output(s)\n[ ] RX disconnection switch\n[ ] DIN connector grounding (pin 2, one end only? cap? what about chassis ground?)\n[ ] EMI ferrite beads on I/O lines?\n\n[X] 12 V connector (incl. GND)? Just use Arduino barrel jack.\n\n[Y] Reset switch\n[Y] MIDI THRU circuitry (buffer)\n[Y] Self-test button\n[Y] Latency control potentiometer\n[Y] LED + resistor on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"
Changed lines of the file:
@@
 LIBS:contrib
 LIBS:valves
+LIBS:dips-s
 LIBS:MIDI_Shield-cache
 EELAYER 25 0
@@
 $EndComp
 $Comp
-L GND #PWR01
+L GND #PWR6
 U 1 1 56E34C2C
 P 7400 4500
-F 0 "#PWR01" H 7400 4500 30  0001 C CNN
+F 0 "#PWR6" H 7400 4500 30  0001 C CNN
 F 1 "GND" H 7400 4430 30  0001 C CNN
 F 2 "" H 7400 4500 60  0000 C CNN
@@
 	1    0    0    -1
 $EndComp
-Wire Wire Line
-	3950 4600 3900 4600
-Wire Wire Line
-	3950 4700 3900 4700
-Wire Wire Line
-	3950 4800 3900 4800
-Wire Wire Line
-	3950 4900 3900 4900
-Text Label 3950 4900 0    60   ~ 0
+Text Label 3900 5600 0    60   ~ 0
 MIDI_CH_1x
-Text Label 3950 4800 0    60   ~ 0
+Text Label 3900 5500 0    60   ~ 0
 MIDI_CH_2x
-Text Label 3950 4700 0    60   ~ 0
+Text Label 3900 5400 0    60   ~ 0
 MIDI_CH_4x
-Text Label 3950 4600 0    60   ~ 0
+Text Label 3900 5300 0    60   ~ 0
 MIDI_CH_8x
 Text Label 2000 4800 2    60   ~ 0
@@
 Text Label 3900 4300 0    60   ~ 0
 GND
-NoConn ~ 3900 5700
 NoConn ~ 2000 4700
 Text Label 2000 5100 2    60   ~ 0
 +12V
 NoConn ~ 3900 4200
-Text Label 3900 5500 0    60   ~ 0
+Text Label 2000 5800 2    60   ~ 0
 SELF_TEST
 $Comp
-L GND #PWR02
+L GND #PWR3
 U 1 1 56E493E9
 P 4600 1850
-F 0 "#PWR02" H 4600 1850 30  0001 C CNN
+F 0 "#PWR3" H 4600 1850 30  0001 C CNN
 F 1 "GND" H 4600 1780 30  0001 C CNN
 F 2 "" H 4600 1850 60  0000 C CNN
@@
 $EndComp
 $Comp
-L GND #PWR03
+L GND #PWR8
 U 1 1 56E4E625
 P 10100 3650
-F 0 "#PWR03" H 10100 3650 30  0001 C CNN
+F 0 "#PWR8" H 10100 3650 30  0001 C CNN
 F 1 "GND" H 10100 3580 30  0001 C CNN
 F 2 "" H 10100 3650 60  0000 C CNN
@@
 NoConn ~ 2000 5600
 NoConn ~ 2000 5700
-NoConn ~ 2000 5800
-NoConn ~ 3900 4500
-NoConn ~ 3900 5100
-NoConn ~ 3900 5200
-NoConn ~ 3900 5300
-NoConn ~ 3900 5400
-NoConn ~ 3900 5600
 Wire Wire Line
 	3050 1450 3350 1450
@@
 	4600 1050 4600 950
 Text Notes 6800 2050 0    60   ~ 0
-TODO:\n\n[ ] Servo output(s)\n[ ] MOSFET output(s)\n[ ] RX disconnection switch\n[ ] DIN connector grounding (pin 2, one end only? cap? what about chassis ground?)\n[ ] EMI ferrite beads on I/O lines?\n\n[X] 12 V connector (incl. GND)? Just use Arduino barrel jack.\n\n[Y] Reset switch\n[Y] MIDI THRU circuitry (buffer)\n[Y] Self-test button\n[Y] Latency control potentiometer\n[Y] LED + resistor on Pin 13\n
+TODO:\n\n[ ] Servo output(s)\n[ ] MOSFET output(s)\n[ ] RX disconnection switch\n[ ] DIN connector grounding (pin 2, one end only? cap? what about chassis ground?)\n[ ] EMI ferrite beads on I/O lines?\n[ ] Polarised SIL connectors for MIDI I/O\n\n[X] 12 V connector (incl. GND)? Just use Arduino barrel jack.\n\n[Y] Reset switch\n[Y] MIDI THRU circuitry (buffer)\n[Y] Self-test button\n[Y] Latency control potentiometer\n[Y] LED + resistor on Pin 13\n
 Text Label 5100 1550 0    60   ~ 0
 MIDI_IN_TTL
@@
 MIDI thru
 $Comp
-L SW_PUSHBUTTON SW?
+L SW_PUSHBUTTON SW3
 U 1 1 572AEBD4
 P 9600 4150
-F 0 "SW?" H 9450 4260 50  0000 C CNN
+F 0 "SW3" H 9450 4260 50  0000 C CNN
 F 1 "SW_PUSHBUTTON" H 9600 4070 50  0000 C CNN
 F 2 "" H 9600 4150 60  0000 C CNN
@@
 $EndComp
 $Comp
-L GND #PWR?
+L GND #PWR9
 U 1 1 572AEBDA
 P 10100 4400
-F 0 "#PWR?" H 10100 4400 30  0001 C CNN
+F 0 "#PWR9" H 10100 4400 30  0001 C CNN
 F 1 "GND" H 10100 4330 30  0001 C CNN
 F 2 "" H 10100 4400 60  0000 C CNN
@@
 LATENCY_ADJ
 $Comp
-L LED D?
+L LED D2
 U 1 1 572AED85
 P 7300 5550
-F 0 "D?" H 7300 5650 50  0000 C CNN
+F 0 "D2" H 7300 5650 50  0000 C CNN
 F 1 "LED" H 7300 5450 50  0000 C CNN
 F 2 "" H 7300 5550 60  0000 C CNN
@@
 $EndComp
 $Comp
-L R R?
+L R R5
 U 1 1 572AEEB8
 P 7300 5100
-F 0 "R?" V 7380 5100 40  0000 C CNN
+F 0 "R5" V 7380 5100 40  0000 C CNN
 F 1 "1K" V 7307 5101 40  0000 C CNN
 F 2 "" V 7230 5100 30  0000 C CNN
@@
 $EndComp
 $Comp
-L GND #PWR?
+L GND #PWR5
 U 1 1 572AEF85
 P 7300 5800
-F 0 "#PWR?" H 7300 5800 30  0001 C CNN
+F 0 "#PWR5" H 7300 5800 30  0001 C CNN
 F 1 "GND" H 7300 5730 30  0001 C CNN
 F 2 "" H 7300 5800 60  0000 C CNN
@@
 	7300 5800 7300 5750
 $Comp
-L POT RV?
+L POT RV1
 U 1 1 572AF20F
 P 9500 5250
-F 0 "RV?" H 9500 5150 50  0000 C CNN
+F 0 "RV1" H 9500 5150 50  0000 C CNN
 F 1 "10K" H 9500 5250 50  0000 C CNN
 F 2 "" H 9500 5250 60  0000 C CNN
@@
 +5V
 $Comp
-L GND #PWR?
+L GND #PWR7
 U 1 1 572AF432
 P 9500 5650
-F 0 "#PWR?" H 9500 5650 30  0001 C CNN
+F 0 "#PWR7" H 9500 5650 30  0001 C CNN
 F 1 "GND" H 9500 5580 30  0001 C CNN
 F 2 "" H 9500 5650 60  0000 C CNN
@@
 $EndComp
 $Comp
-L GND #PWR?
+L GND #PWR2
 U 1 1 572AF481
 P 1750 7150
-F 0 "#PWR?" H 1750 7150 30  0001 C CNN
+F 0 "#PWR2" H 1750 7150 30  0001 C CNN
 F 1 "GND" H 1750 7080 30  0001 C CNN
 F 2 "" H 1750 7150 60  0000 C CNN
@@
 TODO: series resistor?
 $Comp
-L +5V #PWR?
+L +5V #PWR1
 U 1 1 572B0054
 P 1700 6400
-F 0 "#PWR?" H 1700 6490 20  0001 C CNN
+F 0 "#PWR1" H 1700 6490 20  0001 C CNN
 F 1 "+5V" H 1700 6490 30  0000 C CNN
 F 2 "" H 1700 6400 60  0000 C CNN
@@
 Do we need all these GND labels?\nWon't the parent Arduino board connect these anyway?
 $Comp
-L GND #PWR?
+L GND #PWR4
 U 1 1 572B0D3F
 P 5500 3300
-F 0 "#PWR?" H 5500 3300 30  0001 C CNN
+F 0 "#PWR4" H 5500 3300 30  0001 C CNN
 F 1 "GND" H 5500 3230 30  0001 C CNN
 F 2 "" H 5500 3300 60  0000 C CNN
@@
 NoConn ~ 1800 1050
 Connection ~ 4600 1550
+Text Label 3900 5700 0    60   ~ 0
+MIDI_OUT_TTL
+Text Label 3900 5200 0    60   ~ 0
+MOSFET_PWM
+Text Label 3900 5100 0    60   ~ 0
+STEPPER_DIR
+Text Label 3900 4900 0    60   ~ 0
+STEPPER_STEP
+Text Label 3900 4800 0    60   ~ 0
+SERVO_1
+Text Label 3900 4700 0    60   ~ 0
+SERVO_2
+Text Label 3900 4600 0    60   ~ 0
+SERVO_3
+Text Label 3900 4500 0    60   ~ 0
+MOSFET
 $EndSCHEMATC

Commit message: Updated MIDI shield schematics
Parts:
- added K?: CONN_3, symbol CONN_3
Connections:
- wire segments 36 -> 38
Changed lines of the file:
@@
 Text Label 3900 4500 0    60   ~ 0
 MOSFET
+$Comp
+L CONN_3 K?
+U 1 1 5746E7A9
+P 6150 4300
+F 0 "K?" V 6100 4300 50  0000 C CNN
+F 1 "CONN_3" V 6200 4300 40  0000 C CNN
+F 2 "" H 6150 4300 60  0000 C CNN
+F 3 "" H 6150 4300 60  0000 C CNN
+	1    6150 4300
+	1    0    0    1
+$EndComp
+$Comp
+L GND #PWR?
+U 1 1 5746E8C7
+P 5750 4450
+F 0 "#PWR?" H 5750 4450 30  0001 C CNN
+F 1 "GND" H 5750 4380 30  0001 C CNN
+F 2 "" H 5750 4450 60  0000 C CNN
+F 3 "" H 5750 4450 60  0000 C CNN
+	1    5750 4450
+	1    0    0    -1
+$EndComp
+Wire Wire Line
+	5800 4400 5750 4400
+Wire Wire Line
+	5750 4400 5750 4450
 $EndSCHEMATC

Commit message: Added MOSFET output, updated PC900V (wrong pinout)
Parts:
- added C?: C, symbol C
- added D?: DIODE, symbol DIODE
- added D?: LED, symbol LED
- added P3: CONN_MOLEX_POWER, xess:xess-MOLEX-8981-04P, symbol CONN_4
- added P? (x2): CONN_MIDI_IN, symbol CONN_2
- added P?: CONN_2, symbol CONN_2
- added Q?: F12N10L, TO220, symbol F12N10L
- added R?: 100K, symbol R
- added R?: 10R, symbol R
- added R?: 1.8K, symbol R
- D1, R1, R2, R3, R4, U1: footprint ~ -> (none)
- K1: renamed from K?; value CONN_3 -> CONN_SERVO_1
- R5: value 1K -> 330R
Connections:
- net labels added: ARDUINO_+5V, GNDPWR
- wire segments 38 -> 64
Other:
- note added: "Ditch MOSFET LED?"
- note added: "TODO:\n\n[ ] Servo output(s)\n[ ] MOSFET output(s)\n[ ] RX disconnection switch\n[ ] DIN connector grounding (pin 2, one end only? cap? what about chassis ground?)\n[ ] EMI ferrite beads on I/O lines?\n[ ] Polarised SIL connectors for MIDI I/O\n[ ] Bypass caps\n[ ] IC power pins\n\n[X] 12 V connector (incl. GND)? Just use Arduino barrel jack.\n\n[Y] Reset switch\n[Y] MIDI THRU circuitry (buffer)\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"
- note removed: "TODO:\n\n[ ] Servo output(s)\n[ ] MOSFET output(s)\n[ ] RX disconnection switch\n[ ] DIN connector grounding (pin 2, one end only? cap? what about chassis ground?)\n[ ] EMI ferrite beads on I/O lines?\n[ ] Polarised SIL connectors for MIDI I/O\n\n[X] 12 V connector (incl. GND)? Just use Arduino barrel jack.\n\n[Y] Reset switch\n[Y] MIDI THRU circuitry (buffer)\n[Y] Self-test button\n[Y] Latency c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"
- moved on the sheet: IC1, K1, R2, R3, R4, R5, SW1, SW2, SW3, U1A, U1B

Commit message: Updated PCB layout
Parts:
- D2: footprint (none) -> led:LED-3MM
- D3: renamed from D?; footprint (none) -> led:LED-3MM
- Q1: renamed from Q?; footprint TO220 -> discret:TO220
- SW2: footprint (none) -> dip_sockets:DIP-8__300_ELL
- gave numbers to parts that had none: 8
Changed lines of the file:
@@
 F 0 "SW2" V 7850 4050 60  0000 C CNN
 F 1 "DIPS_04" V 8350 4050 60  0000 C CNN
-F 2 "" H 8100 4050 60  0001 C CNN
+F 2 "dip_sockets:DIP-8__300_ELL" H 8100 4050 60  0001 C CNN
 F 3 "" H 8100 4050 60  0000 C CNN
 	1    8100 4050
@@
 F 0 "R1" V 2880 1450 40  0000 C CNN
 F 1 "220R" V 2807 1451 40  0000 C CNN
-F 2 "" V 2730 1450 30  0000 C CNN
+F 2 "" V 2730 1450 30  0001 C CNN
 F 3 "~" H 2800 1450 30  0000 C CNN
 	1    2800 1450
@@
 F 0 "D1" H 3150 1750 40  0000 C CNN
 F 1 "1N914" H 3150 1550 40  0000 C CNN
-F 2 "" H 3150 1650 60  0000 C CNN
+F 2 "" H 3150 1650 60  0001 C CNN
 F 3 "~" H 3150 1650 60  0000 C CNN
 	1    3150 1650
@@
 F 0 "R2" V 4680 1400 40  0000 C CNN
 F 1 "280R" V 4607 1401 40  0000 C CNN
-F 2 "" V 4530 1400 30  0000 C CNN
+F 2 "" V 4530 1400 30  0001 C CNN
 F 3 "~" H 4600 1400 30  0000 C CNN
 	1    4600 1400
@@
 F 0 "R3" V 3330 2800 40  0000 C CNN
 F 1 "220R" V 3257 2801 40  0000 C CNN
-F 2 "" V 3180 2800 30  0000 C CNN
+F 2 "" V 3180 2800 30  0001 C CNN
 F 3 "~" H 3250 2800 30  0000 C CNN
 	1    3250 2800
@@
 F 0 "R4" V 3330 3000 40  0000 C CNN
 F 1 "220R" V 3257 3001 40  0000 C CNN
-F 2 "" V 3180 3000 30  0000 C CNN
+F 2 "" V 3180 3000 30  0001 C CNN
 F 3 "~" H 3250 3000 30  0000 C CNN
 	1    3250 3000
@@
 F 0 "U1" H 2700 3100 40  0000 C CNN
 F 1 "74HC14" H 2750 2900 40  0000 C CNN
-F 2 "" H 2550 3000 60  0000 C CNN
+F 2 "" H 2550 3000 60  0001 C CNN
 F 3 "~" H 2550 3000 60  0000 C CNN
 	2    2550 3000
@@
 F 0 "U1" H 1800 3100 40  0000 C CNN
 F 1 "74HC14" H 1850 2900 40  0000 C CNN
-F 2 "" H 1650 3000 60  0000 C CNN
+F 2 "" H 1650 3000 60  0001 C CNN
 F 3 "~" H 1650 3000 60  0000 C CNN
 	1    1650 3000
@@
 F 0 "D2" H 8000 5650 50  0000 C CNN
 F 1 "LED" H 8000 5450 50  0000 C CNN
-F 2 "" H 8000 5550 60  0001 C CNN
+F 2 "led:LED-3MM" H 8000 5550 60  0001 C CNN
 F 3 "" H 8000 5550 60  0000 C CNN
 	1    8000 5550
@@
 $EndComp
 $Comp
-L GND #PWR?
+L GND #PWR011
 U 1 1 574F9DA1
 P 6400 3050
-F 0 "#PWR?" H 6400 3050 30  0001 C CNN
+F 0 "#PWR011" H 6400 3050 30  0001 C CNN
 F 1 "GND" H 6400 2980 30  0001 C CNN
 F 2 "" H 6400 3050 60  0000 C CNN
@@
 +5V
 $Comp
-L CONN_2 P?
+L CONN_2 P4
 U 1 1 574FB495
 P 2050 1650
-F 0 "P?" V 2000 1650 40  0000 C CNN
+F 0 "P4" V 2000 1650 40  0000 C CNN
 F 1 "CONN_MIDI_IN" V 2100 1650 40  0000 C CNN
-F 2 "" H 2050 1650 60  0000 C CNN
+F 2 "" H 2050 1650 60  0001 C CNN
 F 3 "" H 2050 1650 60  0000 C CNN
 	1    2050 1650
@@
 	1850 1750 2500 1750
 $Comp
-L CONN_2 P?
+L CONN_2 P5
 U 1 1 574FC28D
 P 3950 2900
-F 0 "P?" V 3900 2900 40  0000 C CNN
+F 0 "P5" V 3900 2900 40  0000 C CNN
 F 1 "CONN_MIDI_IN" V 4000 2900 40  0000 C CNN
-F 2 "" H 3950 2900 60  0000 C CNN
+F 2 "" H 3950 2900 60  0001 C CNN
 F 3 "" H 3950 2900 60  0000 C CNN
 	1    3950 2900
@@
 Connection ~ 2400 1750
 $Comp
-L GNDPWR #PWR?
+L GNDPWR #PWR012
 U 1 1 574FC8DB
 P 5500 3350
-F 0 "#PWR?" H 5500 3400 40  0001 C CNN
+F 0 "#PWR012" H 5500 3400 40  0001 C CNN
 F 1 "GNDPWR" H 5500 3270 40  0000 C CNN
 F 2 "" H 5500 3350 60  0000 C CNN
@@
 	3350 1450 3350 1550
 $Comp
-L C C?
+L C C1
 U 1 1 574FCB0A
 P 4300 1400
-F 0 "C?" H 4300 1500 40  0000 L CNN
+F 0 "C1" H 4300 1500 40  0000 L CNN
 F 1 "C" H 4306 1315 40  0000 L CNN
-F 2 "" H 4338 1250 30  0000 C CNN
+F 2 "" H 4338 1250 30  0001 C CNN
 F 3 "" H 4300 1400 60  0000 C CNN
 	1    4300 1400
@@
 Connection ~ 4300 1750
 $Comp
-L F12N10L Q?
+L F12N10L Q1
 U 1 1 574FDEDF
 P 6250 6300
-F 0 "Q?" H 6250 6152 40  0000 R CNN
+F 0 "Q1" H 6250 6152 40  0000 R CNN
 F 1 "F12N10L" H 6250 6450 40  0000 R CNN
-F 2 "TO220" H 6150 6400 25  0000 C CIN
+F 2 "discret:TO220" H 6150 6400 25  0000 C CIN
 F 3 "" H 6250 6300 60  0000 C CNN
 	1    6250 6300
@@
 $EndComp
 $Comp
-L R R?
+L R R8
 U 1 1 574FDFF7
 P 6000 6650
-F 0 "R?" V 6080 6650 40  0000 C CNN
+F 0 "R8" V 6080 6650 40  0000 C CNN
 F 1 "100K" V 6007 6651 40  0000 C CNN
-F 2 "" V 5930 6650 30  0000 C CNN
+F 2 "" V 5930 6650 30  0001 C CNN
 F 3 "" H 6000 6650 30  0000 C CNN
 	1    6000 6650
@@
 $EndComp
 $Comp
-L R R?
+L R R6
 U 1 1 574FE10C
 P 5700 6350
-F 0 "R?" V 5780 6350 40  0000 C CNN
+F 0 "R6" V 5780 6350 40  0000 C CNN
 F 1 "10R" V 5707 6351 40  0000 C CNN
-F 2 "" V 5630 6350 30  0000 C CNN
+F 2 "" V 5630 6350 30  0001 C CNN
 F 3 "" H 5700 6350 30  0000 C CNN
 	1    5700 6350
@@
 $EndComp
 $Comp
-L GND #PWR?
+L GND #PWR013
 U 1 1 574FE201
 P 6000 7000
-F 0 "#PWR?" H 6000 7000 30  0001 C CNN
+F 0 "#PWR013" H 6000 7000 30  0001 C CNN
 F 1 "GND" H 6000 6930 30  0001 C CNN
 F 2 "" H 6000 7000 60  0000 C CNN
@@
 $EndComp
 $Comp
-L GND #PWR?
+L GND #PWR014
 U 1 1 574FE290
 P 6350 7000
-F 0 "#PWR?" H 6350 7000 30  0001 C CNN
+F 0 "#PWR014" H 6350 7000 30  0001 C CNN
 F 1 "GND" H 6350 6930 30  0001 C CNN
 F 2 "" H 6350 7000 60  0000 C CNN
@@
 MOSFET_PWM
 $Comp
-L CONN_2 P?
+L CONN_2 P6
 U 1 1 574FE4C5
 P 6700 5800
-F 0 "P?" V 6650 5800 40  0000 C CNN
+F 0 "P6" V 6650 5800 40  0000 C CNN
 F 1 "CONN_2" V 6750 5800 40  0000 C CNN
-F 2 "" H 6700 5800 60  0000 C CNN
+F 2 "" H 6700 5800 60  0001 C CNN
 F 3 "" H 6700 5800 60  0000 C CNN
 	1    6700 5800
@@
 $EndComp
 $Comp
-L DIODE D?
+L DIODE D4
 U 1 1 574FE5C6
 P 6150 5800
-F 0 "D?" H 6150 5900 40  0000 C CNN
+F 0 "D4" H 6150 5900 40  0000 C CNN
 F 1 "DIODE" H 6150 5700 40  0000 C CNN
-F 2 "" H 6150 5800 60  0000 C CNN
+F 2 "" H 6150 5800 60  0001 C CNN
 F 3 "" H 6150 5800 60  0000 C CNN
 	1    6150 5800
@@
 +12V
 $Comp
-L LED D?
+L LED D3
 U 1 1 574FE85B
 P 5800 5800
-F 0 "D?" H 5800 5900 50  0000 C CNN
+F 0 "D3" H 5800 5900 50  0000 C CNN
 F 1 "LED" H 5800 5700 50  0000 C CNN
-F 2 "" H 5800 5800 60  0000 C CNN
+F 2 "led:LED-3MM" H 5800 5800 60  0001 C CNN
 F 3 "" H 5800 5800 60  0000 C CNN
 	1    5800 5800
@@
 $EndComp
 $Comp
-L R R?
+L R R7
 U 1 1 574FE958
 P 5800 5350
-F 0 "R?" V 5880 5350 40  0000 C CNN
+F 0 "R7" V 5880 5350 40  0000 C CNN
 F 1 "1.8K" V 5807 5351 40  0000 C CNN
-F 2 "" V 5730 5350 30  0000 C CNN
+F 2 "" V 5730 5350 30  0001 C CNN
 F 3 "" H 5800 5350 30  0000 C CNN
 	1    5800 5350

Commit message: - Enlarged page size to A3 and rearranged things a bit  - Added unused hex inverter units in order to ground the inputs  - Refactored 12 V to use a proper power pin  - Added LED for 12 V power  - Relabelled built-in LED on pin 13  - Added servo decoupling cap  - Added additional servo outputs
Parts:
- added C?: 100nF, symbol C
- added D?: LED_PWR_12V, led:LED-3MM, symbol LED
- added R?: 1.8K, symbol R
- added unit 3 of U1
- added unit 4 of U1
- added unit 5 of U1
- added unit 6 of U1
Connections:
- net labels added: LED_BUILTIN
- net labels removed: LED
- wire segments 64 -> 88
- no-connect marks 10 -> 14
Other:
- note added: ""All unused inputs of the device must be held at VCC or GND to ensure proper device operation.""
- note added: "+12V Power LED"
- note added: "Connect cable shield to chassis ground at entry, a la balanced audio cable? The spec says to connect at one end only!"
- note added: "MIDI channel selection"
- note added: "NOTE: the Arduino has a voltage regulator that takes 7-12 V (recommended range) and provides regulated +5 V for powering the board. We also have a +5 V supply from the ATX power supply. We need to distinguish between these, so let's call them ATX+12V, ATX+5V, and ARDUINO+5V."
- note added: "TODO: filter caps, fuses, ..."
- note added: "TODO: use 3.3 V for ADC reference since it's usually better regulated?"
- note added: "Unused hex inverter units:"
- moved on the sheet: D4, K1, P3, P5, P6, Q1, R3, R4, R5, R6, R7, R8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

Commit message: - Relabelled/refactored +5V. The idea is to supply the (noisy) servo motors from ATX +5V directly, and power the Arduino from +12V. The Arduino's regulated +5V will then be used for any logic power, such as the PC900V and the hex inverter.  - Added power, ground, and decoupling for the HC14 chip.
Parts:
- added C?: 100nF, symbol C
Connections:
- net labels added: +5V_LOGIC
- net labels removed: ARDUINO_+5V
- wire segments 88 -> 72
Other:
- note added: "NOTE: the Arduino has a voltage regulator that takes 7-12 V (recommended range) and provides regulated +5 V for powering the board.\nWe also have a +5 V supply from the ATX power supply.\nWe need to distinguish between these, so let's call them ATX+12V, ATX+5V, and ARDUINO+5V."
- note added: "Use ATX +5V for powering only the servo motors? And regulated Arduino +5V for logic only."
- note removed: "NOTE: the Arduino has a voltage regulator that takes 7-12 V (recommended range) and provides regulated +5 V for powering the board. We also have a +5 V supply from the ATX power supply. We need to distinguish between these, so let's call them ATX+12V, ATX+5V, and ARDUINO+5V."
- moved on the sheet: D1, IC1, P3, P4, R1, R2, R?
