File: Projects/2016/MIDIBots/kicad/MIDI_Shield.sch (KiCad schematic (older format))
At the start: 71 parts, among them IC1 PC900V, K1 SRVO1, K2 SRVO2, K3 SRVO3, P1 MIDI_IN, P10 A3, P11 A4, P12 AUX_12V, P13 AUX_12V, P14 AUX_5V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

Commit message: Tidied up PCB footprint labels and moved to visible silkscreen layer
Parts:
- R1, R10, R11, R12, R13, R14, R15, R16, R17, R18, R19, R2, R3, R4, R5, R6, R7, R8, R9: footprint discret:R4-LARGE_PADS -> Discret:R4-LARGE_PADS

Commit message: Some fluffing around with DIP packages; resolved, I think, by using the footprints I saved into the infomechatronics.pretty library
Parts:
- added P?: AD3, symbol CONN_01X01
- added P?: AD4, symbol CONN_01X01
- added P? (x2): GND, symbol CONN_01X01
Connections:
- net labels added: AD3, AD4
- wire segments 139 -> 143
- no-connect marks 14 -> 12
Other:
- note added: "Additional I/O pins:"
Changed lines of the file:
@@
 Wire Wire Line
 	14400 6200 14150 6200
-NoConn ~ 1450 7850
-NoConn ~ 1450 7950
 Wire Wire Line
 	3750 1600 4000 1600
@@
 Wire Wire Line
 	10200 8100 10200 8150
-Text Label 1450 8050 2    60   ~ 0
+Text Label 1450 7850 2    60   ~ 0
 MOSFET_3
-Text Label 1450 8150 2    60   ~ 0
+Text Label 1450 7950 2    60   ~ 0
 MOSFET_4
 $Comp
@@
 	1    0    0    -1
 $EndComp
+Text Label 1450 8050 2    60   ~ 0
+AD3
+Text Label 1450 8150 2    60   ~ 0
+AD4
+Text Label 9350 10200 2    60   ~ 0
+AD3
+Text Label 9350 10350 2    60   ~ 0
+AD4
+Text Notes 9050 10000 0    60   ~ 0
+Additional I/O pins:
+$Comp
+L CONN_01X01 P?
+U 1 1 57539A35
+P 9550 10200
+F 0 "P?" H 9550 10300 50  0000 C CNN
+F 1 "AD3" V 9650 10200 50  0000 C CNN
+F 2 "" H 9550 10200 50  0000 C CNN
+F 3 "" H 9550 10200 50  0000 C CNN
+	1    9550 10200
+	1    0    0    -1
+$EndComp
+$Comp
+L CONN_01X01 P?
+U 1 1 57539CDF
+P 9550 10350
+F 0 "P?" H 9550 10450 50  0000 C CNN
+F 1 "AD4" V 9650 10350 50  0000 C CNN
+F 2 "" H 9550 10350 50  0000 C CNN
+F 3 "" H 9550 10350 50  0000 C CNN
+	1    9550 10350
+	1    0    0    -1
+$EndComp
+$Comp
+L CONN_01X01 P?
+U 1 1 57539EDC
+P 9550 10500
+F 0 "P?" H 9550 10600 50  0000 C CNN
+F 1 "GND" V 9650 10500 50  0000 C CNN
+F 2 "" H 9550 10500 50  0000 C CNN
+F 3 "" H 9550 10500 50  0000 C CNN
+	1    9550 10500
+	1    0    0    -1
+$EndComp
+$Comp
+L CONN_01X01 P?
+U 1 1 57539FE9
+P 9550 10650
+F 0 "P?" H 9550 10750 50  0000 C CNN
+F 1 "GND" V 9650 10650 50  0000 C CNN
+F 2 "" H 9550 10650 50  0000 C CNN
+F 3 "" H 9550 10650 50  0000 C CNN
+	1    9550 10650
+	1    0    0    -1
+$EndComp
+$Comp
+L GND-RESCUE-MIDI_Shield #PWR?
+U 1 1 5753A559
+P 9250 10550
+F 0 "#PWR?" H 9250 10550 30  0001 C CNN
+F 1 "GND" H 9250 10480 30  0001 C CNN
+F 2 "" H 9250 10550 60  0000 C CNN
+F 3 "" H 9250 10550 60  0000 C CNN
+	1    9250 10550
+	1    0    0    -1
+$EndComp
+$Comp
+L GND-RESCUE-MIDI_Shield #PWR?
+U 1 1 5753A654
+P 9250 10700
+F 0 "#PWR?" H 9250 10700 30  0001 C CNN
+F 1 "GND" H 9250 10630 30  0001 C CNN
+F 2 "" H 9250 10700 60  0000 C CNN
+F 3 "" H 9250 10700 60  0000 C CNN
+	1    9250 10700
+	1    0    0    -1
+$EndComp
+Wire Wire Line
+	9250 10700 9250 10650
+Wire Wire Line
+	9250 10650 9350 10650
+Wire Wire Line
+	9250 10550 9250 10500
+Wire Wire Line
+	9250 10500 9350 10500
 $EndSCHEMATC

Commit message: [Y] Remap pins for MOSFET 3 and 4 to make PCB routing easier [Y] Break out remaining Arduino pins (there's only 2!) and put header with a GND in the bottom left corner. [Y] Fixed unexpected mess with use of old DIP socket footprints [Y] Various footprints remapped [Y] SELF_TEST track re-routed slightly
Parts:
- removed P?: AD3, symbol CONN_01X01
- removed P?: AD4, symbol CONN_01X01
- removed P? (x2): GND, symbol CONN_01X01
- added P16: AD3, Pin_Headers:Pin_Header_Straight_1x02, symbol CONN_01X02
- added P17: AD4, Pin_Headers:Pin_Header_Straight_1x02, symbol CONN_01X02
- IC1: footprint dip_sockets:DIP-6__300_ELL -> infomechatronics:DIP-6__300_ELL
- RV1: Label (none) -> LAT_ADJ
- SW2: value DIPS_04 -> MIDI_CH; footprint dip_sockets:DIP-8__300_ELL -> infomechatronics:DIP-8__300_ELL
- U1: footprint dip_sockets:DIP-14__300_ELL -> infomechatronics:DIP-14__300_ELL

Commit message: Relabelled the two left MOSFET output connectors to match their Arduino pins
Parts:
- P10: value A3 -> A1
- P11: value A4 -> A2
Changed lines of the file:
@@
 P 9650 8450
 F 0 "P10" V 9600 8450 40  0000 C CNN
-F 1 "A3" V 9700 8450 40  0000 C CNN
+F 1 "A1" V 9700 8450 40  0000 C CNN
 F 2 "Connect:PINHEAD1-2" H 9650 8450 60  0001 C CNN
 F 3 "" H 9650 8450 60  0000 C CNN
@@
 P 11100 8450
 F 0 "P11" V 11050 8450 40  0000 C CNN
-F 1 "A4" V 11150 8450 40  0000 C CNN
+F 1 "A2" V 11150 8450 40  0000 C CNN
 F 2 "Connect:PINHEAD1-2" H 11100 8450 60  0001 C CNN
 F 3 "" H 11100 8450 60  0000 C CNN

Commit message: Fixed servo pinouts
Connections:
- net +5V: now also K1.2 (PM), K2.2 (PM), K3.2 (PM); no longer K1.3 (P3), K2.3 (P3), K3.3 (P3)
- net SERVO_1: now also K1.3 (P3); no longer K1.2 (PM)
- net SERVO_2: now also K2.3 (P3); no longer K2.2 (PM)
- net SERVO_3: now also K3.3 (P3); no longer K3.2 (PM)
Other:
- moved on the sheet: C3, K2, K3, P8
Changed lines of the file:
@@
 L GND-RESCUE-MIDI_Shield #PWR08
 U 1 1 5746E8C7
-P 8900 5500
-F 0 "#PWR08" H 8900 5500 30  0001 C CNN
-F 1 "GND" H 8900 5430 30  0001 C CNN
-F 2 "" H 8900 5500 60  0000 C CNN
-F 3 "" H 8900 5500 60  0000 C CNN
-	1    8900 5500
+P 8750 5650
+F 0 "#PWR08" H 8750 5650 30  0001 C CNN
+F 1 "GND" H 8750 5580 30  0001 C CNN
+F 2 "" H 8750 5650 60  0000 C CNN
+F 3 "" H 8750 5650 60  0000 C CNN
+	1    8750 5650
 	1    0    0    -1
 $EndComp
@@
 Text Notes 5050 8050 0    60   ~ 0
 Ditch MOSFET LED?\n(if space needed)
-Text Label 8750 5250 2    60   ~ 0
+Text Label 9100 5050 2    60   ~ 0
 SERVO_1
 Wire Wire Line
@@
 L +5V #PWR023
 U 1 1 57516B6C
-P 8900 5050
-F 0 "#PWR023" H 8900 5140 20  0001 C CNN
-F 1 "+5V" H 8900 5140 30  0000 C CNN
-F 2 "" H 8900 5050 60  0000 C CNN
-F 3 "" H 8900 5050 60  0000 C CNN
-	1    8900 5050
+P 8750 5250
+F 0 "#PWR023" H 8750 5340 20  0001 C CNN
+F 1 "+5V" H 8750 5340 30  0000 C CNN
+F 2 "" H 8750 5250 60  0000 C CNN
+F 3 "" H 8750 5250 60  0000 C CNN
+	1    8750 5250
 	1    0    0    -1
 $EndComp
@@
 L C-RESCUE-MIDI_Shield C3
 U 1 1 57516E8B
-P 8900 5250
-F 0 "C3" H 8900 5350 40  0000 L CNN
-F 1 "100nF" H 8906 5165 40  0000 L CNN
-F 2 "Capacitors_ThroughHole:C_Rect_L7_W2.5_P5" H 8938 5100 30  0001 C CNN
-F 3 "" H 8900 5250 60  0000 C CNN
-	1    8900 5250
+P 8750 5450
+F 0 "C3" H 8750 5550 40  0000 L CNN
+F 1 "100nF" H 8756 5365 40  0000 L CNN
+F 2 "Capacitors_ThroughHole:C_Rect_L7_W2.5_P5" H 8788 5300 30  0001 C CNN
+F 3 "" H 8750 5450 60  0000 C CNN
+	1    8750 5450
 	1    0    0    -1
 $EndComp
 Wire Wire Line
 	9100 5050 9100 5150
-Wire Wire Line
-	9100 5050 8900 5050
-Wire Wire Line
-	9100 5350 9100 5450
-Wire Wire Line
-	9100 5450 8900 5450
-Wire Wire Line
-	8900 5450 8900 5500
-Connection ~ 8900 5050
-Connection ~ 8900 5450
+Connection ~ 9100 5050
 Text Notes 8550 1600 0    60   ~ 0
 Power input, filtering, and protection:
@@
 L CONN_3 K2
 U 1 1 5751B9D8
-P 9450 5950
-F 0 "K2" V 9400 5950 50  0000 C CNN
-F 1 "SRVO2" V 9500 5950 40  0000 C CNN
-F 2 "Pin_Headers:Pin_Header_Straight_1x03" H 9450 5950 60  0001 C CNN
-F 3 "" H 9450 5950 60  0000 C CNN
-	1    9450 5950
+P 9450 6200
+F 0 "K2" V 9400 6200 50  0000 C CNN
+F 1 "SRVO2" V 9500 6200 40  0000 C CNN
+F 2 "Pin_Headers:Pin_Header_Straight_1x03" H 9450 6200 60  0001 C CNN
+F 3 "" H 9450 6200 60  0000 C CNN
+	1    9450 6200
 	1    0    0    1
 $EndComp
@@
 L GND-RESCUE-MIDI_Shield #PWR028
 U 1 1 5751B9DE
-P 8900 6200
-F 0 "#PWR028" H 8900 6200 30  0001 C CNN
-F 1 "GND" H 8900 6130 30  0001 C CNN
-F 2 "" H 8900 6200 60  0000 C CNN
-F 3 "" H 8900 6200 60  0000 C CNN
-	1    8900 6200
-	1    0    0    -1
-$EndComp
-Text Label 8750 5950 2    60   ~ 0
+P 9100 6400
+F 0 "#PWR028" H 9100 6400 30  0001 C CNN
+F 1 "GND" H 9100 6330 30  0001 C CNN
+F 2 "" H 9100 6400 60  0000 C CNN
+F 3 "" H 9100 6400 60  0000 C CNN
+	1    9100 6400
+	1    0    0    -1
+$EndComp
+Text Label 9100 6000 2    60   ~ 0
 SERVO_2
 Wire Wire Line
-	8750 5950 9100 5950
+	8750 6200 9100 6200
 $Comp
 L +5V #PWR029
 U 1 1 5751B9E6
-P 8900 5750
-F 0 "#PWR029" H 8900 5840 20  0001 C CNN
-F 1 "+5V" H 8900 5840 30  0000 C CNN
-F 2 "" H 8900 5750 60  0000 C CNN
-F 3 "" H 8900 5750 60  0000 C CNN
-	1    8900 5750
-	1    0    0    -1
-$EndComp
-Wire Wire Line
-	9100 5750 9100 5850
-Wire Wire Line
-	9100 5750 8900 5750
-Wire Wire Line
-	9100 6050 9100 6150
-Wire Wire Line
-	9100 6150 8900 6150
-Wire Wire Line
-	8900 6150 8900 6200
-Connection ~ 8900 5750
-Connection ~ 8900 6150
+P 8750 6200
+F 0 "#PWR029" H 8750 6290 20  0001 C CNN
+F 1 "+5V" H 8750 6290 30  0000 C CNN
+F 2 "" H 8750 6200 60  0000 C CNN
+F 3 "" H 8750 6200 60  0000 C CNN
+	1    8750 6200
+	1    0    0    -1
+$EndComp
+Wire Wire Line
+	9100 6000 9100 6100
+Wire Wire Line
+	9100 6300 9100 6400
+Connection ~ 9100 6000
 $Comp
 L CONN_3 K3
 U 1 1 5751BF4B
-P 9450 6650
-F 0 "K3" V 9400 6650 50  0000 C CNN
-F 1 "SRVO3" V 9500 6650 40  0000 C CNN
-F 2 "Pin_Headers:Pin_Header_Straight_1x03" H 9450 6650 60  0001 C CNN
-F 3 "" H 9450 6650 60  0000 C CNN
-	1    9450 6650
+P 9450 6900
+F 0 "K3" V 9400 6900 50  0000 C CNN
+F 1 "SRVO3" V 9500 6900 40  0000 C CNN
+F 2 "Pin_Headers:Pin_Header_Straight_1x03" H 9450 6900 60  0001 C CNN
+F 3 "" H 9450 6900 60  0000 C CNN
+	1    9450 6900
 	1    0    0    1
 $EndComp
@@
 L GND-RESCUE-MIDI_Shield #PWR030
 U 1 1 5751BF51
-P 8900 6900
-F 0 "#PWR030" H 8900 6900 30  0001 C CNN
-F 1 "GND" H 8900 6830 30  0001 C CNN
-F 2 "" H 8900 6900 60  0000 C CNN
-F 3 "" H 8900 6900 60  0000 C CNN
-	1    8900 6900
-	1    0    0    -1
-$EndComp
-Wire Wire Line
-	8750 6650 9100 6650
+P 9100 7100
+F 0 "#PWR030" H 9100 7100 30  0001 C CNN
+F 1 "GND" H 9100 7030 30  0001 C CNN
+F 2 "" H 9100 7100 60  0000 C CNN
+F 3 "" H 9100 7100 60  0000 C CNN
+	1    9100 7100
+	1    0    0    -1
+$EndComp
+Wire Wire Line
+	8750 6900 9100 6900
 $Comp
 L +5V #PWR031
 U 1 1 5751BF59
-P 8900 6450
-F 0 "#PWR031" H 8900 6540 20  0001 C CNN
-F 1 "+5V" H 8900 6540 30  0000 C CNN
-F 2 "" H 8900 6450 60  0000 C CNN
-F 3 "" H 8900 6450 60  0000 C CNN
-	1    8900 6450
-	1    0    0    -1
-$EndComp
-Wire Wire Line
-	9100 6450 9100 6550
-Wire Wire Line
-	9100 6450 8900 6450
-Wire Wire Line
-	9100 6750 9100 6850
-Wire Wire Line
-	9100 6850 8900 6850
-Wire Wire Line
-	8900 6850 8900 6900
-Connection ~ 8900 6450
-Connection ~ 8900 6850
-Text Label 8750 6650 2    60   ~ 0
+P 8750 6900
+F 0 "#PWR031" H 8750 6990 20  0001 C CNN
+F 1 "+5V" H 8750 6990 30  0000 C CNN
+F 2 "" H 8750 6900 60  0000 C CNN
+F 3 "" H 8750 6900 60  0000 C CNN
+	1    8750 6900
+	1    0    0    -1
+$EndComp
+Wire Wire Line
+	9100 6700 9100 6800
+Connection ~ 9100 6700
+Text Label 9100 6700 2    60   ~ 0
 SERVO_3
 Text Notes 6150 7700 0    60   ~ 0
@@
 L CONN_2 P8
 U 1 1 5751DBD1
-P 10950 5750
-F 0 "P8" V 10900 5750 40  0000 C CNN
-F 1 "STEPPER" V 11000 5750 40  0000 C CNN
-F 2 "Connect:PINHEAD1-2" H 10950 5750 60  0001 C CNN
-F 3 "" H 10950 5750 60  0000 C CNN
-	1    10950 5750
+P 11250 5050
+F 0 "P8" V 11200 5050 40  0000 C CNN
+F 1 "STEPPER" V 11300 5050 40  0000 C CNN
+F 2 "Connect:PINHEAD1-2" H 11250 5050 60  0001 C CNN
+F 3 "" H 11250 5050 60  0000 C CNN
+	1    11250 5050
 	1    0    0    1
 $EndComp
-Text Label 10600 5850 2    60   ~ 0
+Text Label 10900 5150 2    60   ~ 0
 STEPPER_DIR
-Text Label 10600 5650 2    60   ~ 0
+Text Label 10900 4950 2    60   ~ 0
 STEPPER_STEP
-Text Notes 10000 5450 0    60   ~ 0
+Text Notes 10300 4750 0    60   ~ 0
 Stepper motor output:
 $Comp
@@
 	1    0    0    1
 $EndComp
+Wire Wire Line
+	9100 7100 9100 7000
+Wire Wire Line
+	8750 5650 8750 5600
+Wire Wire Line
+	8750 5600 9100 5600
+Wire Wire Line
+	9100 5600 9100 5350
 $EndSCHEMATC
